Commit message: restructured

File: catkin_ws/src/rover_autonav/urdf/rosbob_v5.xacro (robot description, xacro)
@@ -38,5 +38,5 @@
 			<origin xyz="0 0 0.3429" rpy=" 0 0 ${half_pi}"/>
 			<geometry>
-				<mesh filename="package://rover_autonav/meshes_v2/base_link_armless.STL" />
+				<mesh filename="package://rover_autonav/meshes/base_link_armless.STL" />
 				<!-- <box size="${robot_chassis_length} ${robot_chassis_width} ${robot_chassis_height}"/> -->
 			</geometry>
@@ -57,5 +57,5 @@
 			<origin xyz="0 0 0" rpy="1.5707 0.0 -1.5707"/>
 			<geometry>
-				<mesh filename="package://rover_autonav/meshes_v2/wheel.STL" />
+				<mesh filename="package://rover_autonav/meshes/wheel.STL" />
 				<!-- <cylinder radius="${robot_wheel_radius}" length="${robot_wheel_length}"/> -->
 			</geometry>
@@ -82,5 +82,5 @@
 			<origin xyz="0 0 0" rpy="1.5707 0.0 -1.5707"/>
 			<geometry>
-				<mesh filename="package://rover_autonav/meshes_v2/wheel.STL" />
+				<mesh filename="package://rover_autonav/meshes/wheel.STL" />
 				<!-- <cylinder radius="${robot_wheel_radius}" length="${robot_wheel_length}"/> -->
 			</geometry>
@@ -107,5 +107,5 @@
 			<origin xyz="0 0 0" rpy="1.5707 0.0 -1.5707"/>
 			<geometry>
-				<mesh filename="package://rover_autonav/meshes_v2/wheel.STL" />
+				<mesh filename="package://rover_autonav/meshes/wheel.STL" />
 				<!-- <cylinder radius="${robot_wheel_radius}" length="${robot_wheel_length}"/> -->
 			</geometry>
@@ -132,5 +132,5 @@
 			<origin xyz="0 0 0" rpy="1.5707 0.0 -1.5707"/>
 			<geometry>
-				<mesh filename="package://rover_autonav/meshes_v2/wheel.STL" />
+				<mesh filename="package://rover_autonav/meshes/wheel.STL" />
 				<!-- <cylinder radius="${robot_wheel_radius}" length="${robot_wheel_length}"/> -->
 			</geometry>
