Commit message: cleaned

File: catkin_ws/src/manipulation/description/urdf/arm_world_frame.xacro (robot description, xacro)
@@ -367,5 +367,5 @@
         <origin xyz="0 0 0" rpy="0 0 0"/>
         <geometry>
-          <mesh filename="package://rover_autonav/meshes/d435.dae"/>
+          <mesh filename="package://navigation/description/meshes/d435.dae"/>
         </geometry>
       </visual>

File: catkin_ws/src/navigation/description/urdf/cali.xacro (robot description, xacro)
@@ -3,5 +3,5 @@
        name="ur3e" >
   <!-- MOBILE ROBOT -->
-  <xacro:include filename="$(find rover_autonav)/description/urdf/cali_base.xacro" />
+  <xacro:include filename="$(find navigation)/description/urdf/cali_base.xacro" />
   <!-- ARM -->
   <xacro:include filename="$(find manipulation)/description/urdf/arm.xacro" />

File: catkin_ws/src/navigation/description/urdf/cali_base.xacro (robot description, xacro)
@@ -38,5 +38,5 @@
 			<origin xyz="0 0 0.3429" rpy=" 0 0 ${half_pi}"/>
 			<geometry>
-				<mesh filename="package://rover_autonav/description/meshes/base_link_armless.STL" />
+				<mesh filename="package://navigation/description/meshes/base_link_armless.STL" />
 				<!-- <box size="${robot_chassis_length} ${robot_chassis_width} ${robot_chassis_height}"/> -->
 			</geometry>
@@ -57,5 +57,5 @@
 			<origin xyz="0 0 0" rpy="1.5707 0.0 -1.5707"/>
 			<geometry>
-				<mesh filename="package://rover_autonav/description/meshes/wheel.STL" />
+				<mesh filename="package://navigation/description/meshes/wheel.STL" />
 				<!-- <cylinder radius="${robot_wheel_radius}" length="${robot_wheel_length}"/> -->
 			</geometry>
@@ -82,5 +82,5 @@
 			<origin xyz="0 0 0" rpy="1.5707 0.0 -1.5707"/>
 			<geometry>
-				<mesh filename="package://rover_autonav/description/meshes/wheel.STL" />
+				<mesh filename="package://navigation/description/meshes/wheel.STL" />
 				<!-- <cylinder radius="${robot_wheel_radius}" length="${robot_wheel_length}"/> -->
 			</geometry>
@@ -107,5 +107,5 @@
 			<origin xyz="0 0 0" rpy="1.5707 0.0 -1.5707"/>
 			<geometry>
-				<mesh filename="package://rover_autonav/description/meshes/wheel.STL" />
+				<mesh filename="package://navigation/description/meshes/wheel.STL" />
 				<!-- <cylinder radius="${robot_wheel_radius}" length="${robot_wheel_length}"/> -->
 			</geometry>
@@ -132,5 +132,5 @@
 			<origin xyz="0 0 0" rpy="1.5707 0.0 -1.5707"/>
 			<geometry>
-				<mesh filename="package://rover_autonav/description/meshes/wheel.STL" />
+				<mesh filename="package://navigation/description/meshes/wheel.STL" />
 				<!-- <cylinder radius="${robot_wheel_radius}" length="${robot_wheel_length}"/> -->
 			</geometry>
@@ -183,5 +183,5 @@
 			<origin xyz="0 0 0" rpy="0 0 0"/>
 			<geometry>
-				<mesh filename="package://rover_autonav/description/meshes/hokuyo.dae"/>
+				<mesh filename="package://navigation/description/meshes/hokuyo.dae"/>
 			</geometry>
 		</visual>
@@ -315,4 +315,4 @@
 	</gazebo>
 	<!-- Motor, Camera and Lidar Simulation -->
-	<xacro:include filename="$(find rover_autonav)/description/urdf/cali_base.gazebo" />
+	<xacro:include filename="$(find navigation)/description/urdf/cali_base.gazebo" />
 </robot>
